File: circuit/circuit.kicad_sch (KiCad schematic)
At the start: 1 part, among them U1 Pico

Commit message: .
Parts:
- removed U1: Pico, RPi_Pico:RPi_Pico_SMD_TH, symbol MCU_RaspberryPi_and_Boards:Pico
- added BZ1: Buzzer, symbol Device:Buzzer
- added D1, D2: 1N4148, Diode_THT:D_DO-35_SOD27_P7.62mm_Horizontal, symbol Diode:1N4148
- added J1: Micro_SD_Card, symbol Connector:Micro_SD_Card
- added J2: USB-C Power, symbol Connector:USB_C_Receptacle_PowerOnly_6P
- added J4: VGA, symbol Connector:DE15_Receptacle_HighDensity
- added J?: FTDI cable, symbol Connector_Generic:Conn_01x06
- added R1, R2, R3, R4, R5, R6, R7: 220, symbol Device:R
- added RV1: Trim 200, symbol Device:R_Potentiometer_Trim
- added SW1: RESET, symbol Switch:SW_Push
- added U1: ESP-PSRAM32, Package_SO:SOIC-8_3.9x4.9mm_P1.27mm, symbol Memory_RAM:ESP-PSRAM32
- added U2: TXB0104PW, Package_SO:TSSOP-14_4.4x5mm_P0.65mm, symbol Logic_LevelTranslator:TXB0104PW
- added U7: Pico, RPi_Pico:RPi_Pico_SMD_TH, symbol MCU_RaspberryPi_and_Boards:Pico
Connections:
- new net: SW1.1, U7.30 (RUN)
- new net: D2.2 (A), J4.1, R5.2
- new net: R1.2, R2.1, R3.1, R4.2
- new net: BZ1.1 (-), U7.20 (GPIO15)
- new net: J4.2, R6.2
- new net: D1.2 (A), J4.3, R7.2
- new net: U2.10 (B4), U7.5 (GPIO3)
- new net: U2.11 (B3), U7.4 (GPIO2)
- new net: U2.12 (B2), U7.2 (GPIO1)
- new net: U2.13 (B1), U7.1 (GPIO0)
- new net +3.3V: J1.4 (VDD), U1.8 (VCC), U2.14 (VCCB), U7.36 (3V3)
- new net +5V: J2.A9 (VBUS), J2.B9 (VBUS), J?.3 (Pin_3), U2.1 (VCCA), U7.39 (VSYS)
- new net BLUE: R7.1, U7.24 (GPIO18)
- new net CTS: J?.2 (Pin_2), U2.4 (A3)
- new net DTR: J?.6 (Pin_6), U2.5 (A4)
- new net GND: BZ1.2 (+), D1.1 (K), D2.1 (K), J1.6 (VSS), J2.A12 (GND), J2.B12 (GND), J4.10, J4.5, J4.6, J4.7, J4.8, J?.1 (Pin_1), R4.1, RV1.2, SW1.2, U1.4 (VSS), U2.7 (GND), U7.23 (GND)
- new net GREEN0: R1.1, U7.26 (GPIO20)
- new net GREEN1: R2.2, R3.2, R6.1, RV1.1, U7.25 (GPIO19)
- new net HSYNC: J4.13, U7.21 (GPIO16)
- new net MISO: J1.7 (DAT0), U1.2 (SO/SIO), U7.16 (GPIO12)
- new net MOSI: J1.3 (CMD), U1.5 (SI/SIO), U7.15 (GPIO11)
- new net PCRX: J?.5 (Pin_5), U2.3 (A2)
- new net PCTX: J?.4 (Pin_4), U2.2 (A1)
- new net RAM_CS: U1.1 (~{CE}), U7.12 (GPIO9)
- new net RED: R5.1, U7.27 (GPIO21)
- new net SCK: J1.5 (CLK), U1.6 (SCLK), U7.14 (GPIO10)
- new net SD_CS: J1.2 (DAT3/CD), U7.17 (GPIO13)
- new net VSYNC: J4.14, U7.22 (GPIO17)
- no-connect marks 0 -> 12

Commit message: .
Parts:
- removed J?: FTDI cable, symbol Connector_Generic:Conn_01x06
- removed U2: TXB0104PW, Package_SO:TSSOP-14_4.4x5mm_P0.65mm, symbol Logic_LevelTranslator:TXB0104PW
- added D3: LED, symbol Device:LED
- added R8: R, symbol Device:R
Connections:
- net +3.3V: now also D3.2 (A)
- net at U7.1 (GPIO0): now also R8.2
- new net: D3.1 (K), R8.1
Other:
- moved on the sheet: J2

Commit message: .
Parts:
- removed J1: Micro_SD_Card, symbol Connector:Micro_SD_Card
- added J3: Micro_SD_Card_Det1, symbol Connector:Micro_SD_Card_Det1
- added R9: 10k, symbol Device:R
Connections:
- net +3.3V: now also J3.3 (CMD), R9.2
- net GND: now also J3.5 (CLK)
- net MISO: now also J3.6 (VSS)
- net MOSI: now also J3.2 (DAT3/CD)
- net SCK: now also J3.4 (VDD)
- net SD_CS: now also J3.1 (DAT2)
- net CD: now reaches U7.19 (GPIO14)
- net CD: now also J3.9 (DET), R9.1
Changed lines of the file:
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@@
   (junction (at 100.965 143.51) (diameter 0) (color 0 0 0 0)
+  )
+  (junction (at 207.01 70.485) (diameter 0) (color 0 0 0 0)
   )
   (junction (at 83.82 156.21) (diameter 0) (color 0 0 0 0)
@@
   (no_connect (at 120.015 146.05))
   (no_connect (at 229.87 106.68))
-  (no_connect (at 227.965 45.085))
+  (no_connect (at 227.965 65.405))
   (no_connect (at 227.965 62.865))
   (no_connect (at 50.165 88.9))
@@
     (stroke (width 0) (type default))
   )
+  (wire (pts (xy 207.01 70.485) (xy 227.965 70.485))
+    (stroke (width 0) (type default))
+  )
   (wire (pts (xy 214.63 99.06) (xy 229.87 99.06))
     (stroke (width 0) (type default))
@@
     (stroke (width 0) (type default))
   )
+  (wire (pts (xy 207.01 55.245) (xy 207.01 59.055))
+    (stroke (width 0) (type default))
+  )
   (wire (pts (xy 214.63 101.6) (xy 229.87 101.6))
     (stroke (width 0) (type default))
@@
     (stroke (width 0) (type default))
   )
+  (wire (pts (xy 207.01 66.675) (xy 207.01 70.485))
+    (stroke (width 0) (type default))
+  )
+  (wire (pts (xy 201.93 70.485) (xy 207.01 70.485))
+    (stroke (width 0) (type default))
+  )
   (wire (pts (xy 100.965 148.59) (xy 104.775 148.59))
     (stroke (width 0) (type default))
@@
     (stroke (width 0) (type default))
   )
-  (wire (pts (xy 224.155 57.785) (xy 224.155 71.12))
+  (wire (pts (xy 224.155 57.785) (xy 224.155 76.2))
     (stroke (width 0) (type default))
   )
@@
     (stroke (width 0) (type default))
   )
+  (wire (pts (xy 123.19 95.25) (xy 138.43 95.25))
+    (stroke (width 0) (type default))
+  )
   (wire (pts (xy 100.965 166.37) (xy 100.965 168.91))
     (stroke (width 0) (type default))
@@
   (wire (pts (xy 60.96 160.02) (xy 60.96 162.56))
     (stroke (width 0) (type default))
+  )
+  (label "CD" (at 201.93 70.485 0) (fields_autoplaced)
+    (effects (font (size 1.27 1.27)) (justify left bottom))
   )
   (label "VSYNC" (at 130.175 161.29 180) (fields_autoplaced)
@@
     (effects (font (size 1.27 1.27)) (justify left bottom))
   )
+  (label "CD" (at 123.19 95.25 0) (fields_autoplaced)
+    (effects (font (size 1.27 1.27)) (justify left bottom))
+  )
   (label "HSYNC" (at 189.23 97.79 180) (fields_autoplaced)
     (effects (font (size 1.27 1.27)) (justify right bottom))
@@
         (path "/0a6b6e71-7152-4192-b04d-e2f91e81ba3a"
           (reference "R5") (unit 1)
+        )
+      )
+    )
+  )
+  (symbol (lib_id "power:+3.3V") (at 207.01 55.245 0) (mirror y) (unit 1)
+    (in_bom yes) (on_board yes) (dnp no)
+    (property "Reference" "#PWR08" (at 207.01 59.055 0)
+      (effects (font (size 1.27 1.27)) hide)
+    )
+    (property "Value" "+3.3V" (at 202.565 53.34 0)
+      (effects (font (size 1.27 1.27)))
+    )
+    (property "Footprint" "" (at 207.01 55.245 0)
+      (effects (font (size 1.27 1.27)) hide)
+    )
+    (property "Datasheet" "" (at 207.01 55.245 0)
+      (effects (font (size 1.27 1.27)) hide)
+    )
+    (pin "1")
+    (instances
+      (project "circuit"
+        (path "/0a6b6e71-7152-4192-b04d-e2f91e81ba3a"
+          (reference "#PWR08") (unit 1)
         )
       )
@@
         (path "/0a6b6e71-7152-4192-b04d-e2f91e81ba3a"
           (reference "#PWR02") (unit 1)
+        )
+      )
+    )
+  )
+  (symbol (lib_id "Device:R") (at 207.01 62.865 180) (unit 1)
+    (in_bom yes) (on_board yes) (dnp no) (fields_autoplaced)
+    (property "Reference" "R9" (at 208.915 61.595 0)
+      (effects (font (size 1.27 1.27)) (justify right))
+    )
+    (property "Value" "10k" (at 208.915 64.135 0)
+      (effects (font (size 1.27 1.27)) (justify right))
+    )
+    (property "Footprint" "" (at 208.788 62.865 90)
+      (effects (font (size 1.27 1.27)) hide)
+    )
+    (property "Datasheet" "~" (at 207.01 62.865 0)
+      (effects (font (size 1.27 1.27)) hide)
+    )
+    (pin "1")
+    (pin "2")
+    (instances
+      (project "circuit"
+        (path "/0a6b6e71-7152-4192-b04d-e2f91e81ba3a"
+          (reference "R9") (unit 1)
         )
       )
@@
     )
   )
-  (symbol (lib_id "power:GND") (at 224.155 71.12 0) (mirror y) (unit 1)
-    (in_bom yes) (on_board yes) (dnp no)
-    (property "Reference" "#PWR06" (at 224.155 77.47 0)
-      (effects (font (size 1.27 1.27)) hide)
-    )
-    (property "Value" "GND" (at 228.6 73.025 0)
-      (effects (font (size 1.27 1.27)))
-    )
-    (property "Footprint" "" (at 224.155 71.12 0)
-      (effects (font (size 1.27 1.27)) hide)
-    )
-    (property "Datasheet" "" (at 224.155 71.12 0)
+  (symbol (lib_id "power:GND") (at 224.155 76.2 0) (mirror y) (unit 1)
+    (in_bom yes) (on_board yes) (dnp no)
+    (property "Reference" "#PWR06" (at 224.155 82.55 0)
+      (effects (font (size 1.27 1.27)) hide)
+    )
+    (property "Value" "GND" (at 228.6 78.105 0)
+      (effects (font (size 1.27 1.27)))
+    )
+    (property "Footprint" "" (at 224.155 76.2 0)
+      (effects (font (size 1.27 1.27)) hide)
+    )
+    (property "Datasheet" "" (at 224.155 76.2 0)
       (effects (font (size 1.27 1.27)) hide)
     )
@@
     )
   )
-  (symbol (lib_id "Connector:Micro_SD_Card") (at 250.825 52.705 0) (unit 1)
-    (in_bom yes) (on_board yes) (dnp no)
-    (property "Reference" "J1" (at 251.46 34.29 0)
-      (effects (font (size 1.27 1.27)))
-    )
-    (property "Value" "Micro_SD_Card" (at 251.46 36.83 0)
-      (effects (font (size 1.27 1.27)))
-    )
-    (property "Footprint" "" (at 280.035 45.085 0)
-      (effects (font (size 1.27 1.27)) hide)
-    )
-    (property "Datasheet" "http://katalog.we-online.de/em/datasheet/693072010801.pdf" (at 250.825 52.705 0)
-      (effects (font (size 1.27 1.27)) hide)
-    )
-    (pin "1")
+  (symbol (lib_id "Connector:Micro_SD_Card_Det1") (at 250.825 57.785 0) (unit 1)
+    (in_bom yes) (on_board yes) (dnp no) (fields_autoplaced)
+    (property "Reference" "J3" (at 251.46 36.83 0)
+      (effects (font (size 1.27 1.27)))
+    )
+    (property "Value" "Micro_SD_Card_Det1" (at 251.46 39.37 0)
+      (effects (font (size 1.27 1.27)))
+    )
+    (property "Footprint" "" (at 302.895 40.005 0)
+      (effects (font (size 1.27 1.27)) hide)
+    )
+    (property "Datasheet" "https://datasheet.lcsc.com/lcsc/2110151630_XKB-Connectivity-XKTF-015-N_C381082.pdf" (at 250.825 55.245 0)
+      (effects (font (size 1.27 1.27)) hide)
+    )
+    (pin "1")
+    (pin "10")
     (pin "2")
     (pin "3")
@@
       (project "circuit"
         (path "/0a6b6e71-7152-4192-b04d-e2f91e81ba3a"
-          (reference "J1") (unit 1)
-        )
-      )
+          (reference "J3") (unit 1)
+        )
+      )

Commit message: .
Parts:
- removed R9: 10k, symbol Device:R
Connections:
- net CD: now also U7.9 (GPIO6); no longer U7.19 (GPIO14)
- net MISO: now also U7.6 (GPIO4); no longer U7.16 (GPIO12)
- net MOSI: now also U7.5 (GPIO3); no longer U7.15 (GPIO11)
- net SCK: now also U7.4 (GPIO2); no longer U7.14 (GPIO10)
- net SD_CS: now also U7.7 (GPIO5); no longer U7.17 (GPIO13)
- net at BZ1.1 (-): now also U7.2 (GPIO1); no longer U7.20 (GPIO15)
